File: Neonest_V_1.3.kicad_pcb (KiCad board)
At the start: 2 copper layers, 75 x 88 mm, 99 parts, among them J3 693071010811, J5 Conn_01x02, J6 Conn_01x05, J7 Conn_01x03, Q1 BC817, Q2 BC817, Q3 STB33N65M2, Q4 BC817, Q5 STB33N65M2, Q6 STB33N65M2, Q7 BC817, U1 LM2596T-5, U2 LM1117-3.3, U3 STM32F103CBTx, Y1 32.678kHz, Y2 8Mhz

Commit message: Minor changes, generated gerber files and submitted
Parts:
- removed TP1, TP2: TestPoint, TestPoint:TestPoint_Pad_D2.5mm
- added JP1: Jumper_2_Bridged, Jumper:SolderJumper-2_P1.3mm_Bridged2Bar_RoundedPad1.0x1.5mm, F.Cu at (159.9, 90.5)
- added SW1: SW_DIP_x01, Button_Switch_THT:SW_PUSH_1P1T_6x3.5mm_H5.0_APEM_MJTP1250, F.Cu at (126.3, 94.8)
- added SW2: SW_DIP_x01, Button_Switch_THT:SW_PUSH_1P1T_6x3.5mm_H5.0_APEM_MJTP1250, F.Cu at (128.1, 122.5)
- added SW3: SW_DIP_x01, Button_Switch_THT:SW_PUSH_1P1T_6x3.5mm_H5.0_APEM_MJTP1250, F.Cu at (144.8, 135.7)
- D7, D8: value STTH2002D -> STTH20R04D
- Q3, Q5, Q6: value STB33N65M2 -> STP80NF70
- R1, R3, R5: value 180k/(1%)0.1W -> 100k/(1%)0.1W
- R2: value 10k/(1%)0.1W -> 22k/(1%)0.1W
- R20: value 0R -> 2R2; footprint Resistor_SMD:R_0603_1608Metric -> Resistor_THT:R_Axial_DIN0204_L3.6mm_D1.6mm_P7.62mm_Horizontal
- R4, R6: value 5.1k/(1%)0.1W -> 22k/(1%)0.1W
- moved REF** 39.0 mm to (150.4, 131.0)
- moved R20 5.39 mm to (146.6, 90.9)
- moved D1 0.48 mm to (123.9, 132.3)
- renumbered BATTERY to J1, YELLOW to J10, GREEN to J11, RED to J12, ADAPTER to J2, TEMP to J4, LCD to J8, HEATER to J9
Connections:
- net /microcontroller/bat_vadc renamed /Microcontroller/bat_vadc
- net /microcontroller/charger_vadc renamed /Microcontroller/charger_vadc
- net /microcontroller/hpad_vadc renamed /Microcontroller/hpad_vadc
- C1 pad 2: GND -> GNDS
- C10 pad 2: GND -> GNDS
- C2 pad 2: GND -> GNDS
- C5 pad 2: GND -> GNDS
- C6 pad 2: GND -> GNDS
- C7 pad 2: GND -> GNDS
- J1 pad 2: BAT -> Net-(J1-Pin_2)
- J2 pad 2: Charger -> Net-(J2-Pin_2)
- R2 pad 2: GND -> GNDS
- R4 pad 2: GND -> GNDS
- R6 pad 2: GND -> GNDS
- U3 pad 8: GND -> GNDS
Routing:
- net GNDS: track 0.00 -> 54.6 mm, vias 0 -> 5
- net Charger: track 108.7 -> 83.0 mm, vias 7 -> 0
- net GND: track 244.3 -> 222.5 mm, vias 41 -> 43
- net Net-(J2-Pin_2): track 0.00 -> 18.1 mm
- net BAT: track 168.1 -> 184.7 mm, vias 12 -> 15
- net Net-(J1-Pin_2): track 0.00 -> 12.1 mm
- net /Load/charge: track 98.2 -> 104.2 mm
- net /Load/charging_pwm: track 87.0 -> 83.8 mm
- net /Load/bat_heating_pwm: track 100.3 -> 97.3 mm
- net /Load/ac_heating_pwm: track 76.5 -> 79.0 mm
- net Net-(Q3-D): track 19.5 -> 17.8 mm
- net Net-(D1-K): track 25.0 -> 23.9 mm
- net Net-(U1-VIN): track 27.4 -> 26.7 mm
- added copper zone on F.Cu, net GNDS
Other:
- board text added: "ADAPTER"
- board text added: "BATTERY"
- board text added: "GREEN"
- board text added: "Gnd"
- board text added: "HEATER"
- board text added: "LCD"
- board text added: "Prog"
- board text added: "RED"
- board text added: "Rx"
- board text added: "TEMP"
- board text added: "Tx"
- board text added: "YELLOW"
