File: mosfet_driver.kicad_sch (KiCad schematic)
At the start: 22 parts, among them J9 Heating pad, Q2 BC817, Q3 STB33N65M2, Q4 BC817, Q5 STB33N65M2, Q6 STB33N65M2, Q7 BC817

Commit message: Formatted schematic and Increased power tracks
Other:
- note added: "Battery sizing Single cell 2600mAH 3.7V lithiu Ion 3P4S(3 serries, 4 in parallel) Total cell configuration 7.8AH 14.8V(16.8V maximum)"
- company: (none) -> Che innovations
- title: (none) -> Neonest v 1.3
Changed lines of the file:
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@@
 (kicad_sch (version 20230121) (generator eeschema)
   (paper "A4")
+  (title_block
+    (title "Neonest v 1.3")
+    (date "2025-08-07")
+    (company "Che innovations")
+  )
   (junction (at 111.76 86.995) (diameter 0) (color 0 0 0 0)
   )
@@
   )
   (text "Heating pad power sources" (at 135.255 26.035 0)
-    (effects (font (size 2.2606 2.2606) italic) (justify left bottom))
+    (effects (font (size 2.2606 2.2606) (thickness 0.4521) bold italic) (justify left bottom))
+  )
+  (text "Battery sizing\nSingle cell 2600mAH\n3.7V lithiu Ion 3P4S(3 serries, 4 in parallel)\nTotal cell configuration 7.8AH 14.8V(16.8V maximum)\n"
+    (at 120.65 170.18 0)
+    (effects (font (size 1.27 1.27)) (justify left bottom))
   )
   (label "charge" (at 92.71 126.365 0) (fields_autoplaced)

Commit message: Few final amendments on sizing and BOM editing
Parts:
- D7, D8: value STTH2002D -> STTH20R04D
- Q3, Q5, Q6: value STB33N65M2 -> STP80NF70
Other:
- note added: "Battery sizing Single cell 2600mAH(12 cells total) 3.7V lithiu Ion 3S4P(3 serries, 4 in parallel) Total cell configuration 10.4AH 14.8V(16.8V maximum)"
- note removed: "Battery sizing Single cell 2600mAH 3.7V lithiu Ion 3P4S(3 serries, 4 in parallel) Total cell configuration 7.8AH 14.8V(16.8V maximum)"
Changed lines of the file:
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@@
     (stroke (width 0) (type default))
   )
-  (text "ST STTH6004W\nLCSC Part :C169788\n" (at 131.445 48.895 0)
+  (text "ST STTH6004W\nLCSC Part :C169788\n" (at 129.286 63.119 0)
     (effects (font (size 1.27 1.27)) (justify left bottom))
   )
@@
     (effects (font (size 2.2606 2.2606) (thickness 0.4521) bold italic) (justify left bottom))
   )
-  (text "Battery sizing\nSingle cell 2600mAH\n3.7V lithiu Ion 3P4S(3 serries, 4 in parallel)\nTotal cell configuration 7.8AH 14.8V(16.8V maximum)\n"
-    (at 120.65 170.18 0)
+  (text "Battery sizing\nSingle cell 2600mAH(12 cells total)\n3.7V lithiu Ion 3S4P(3 serries, 4 in parallel)\nTotal cell configuration 10.4AH 14.8V(16.8V maximum)\n"
+    (at 121.793 142.24 0)
     (effects (font (size 1.27 1.27)) (justify left bottom))
   )
@@
     (in_bom yes) (on_board yes) (dnp no)
     (property "Reference" "Q5" (at 130.302 66.1416 0)
-      (effects (font (size 1.27 1.27)) (justify left) hide)
-    )
-    (property "Value" "STB33N65M2" (at 130.302 68.453 0)
-      (effects (font (size 1.27 1.27)) (justify left) hide)
+      (effects (font (size 1.27 1.27)) (justify left))
+    )
+    (property "Value" "STP80NF70" (at 130.302 68.453 0)
+      (effects (font (size 1.27 1.27)) (justify left))
     )
     (property "Footprint" "Package_TO_SOT_THT:TO-262-3_Vertical" (at 130.175 69.215 0)
@@
       (effects (font (size 1.27 1.27)) (justify right))
     )
-    (property "Value" "STTH2002D" (at 186.055 47.625 90)
+    (property "Value" "STTH20R04D" (at 186.055 47.625 90)
       (effects (font (size 1.27 1.27)) (justify right))
     )
@@
       (effects (font (size 1.27 1.27)) hide)
     )
-    (pin "1")
-    (pin "2")
-    (pin "3")
+    (pin "3")
+    (pin "1")
+    (pin "2")
     (instances
       (project "Neonest_V_1.3"
@@
     (in_bom yes) (on_board yes) (dnp no)
     (property "Reference" "Q6" (at 168.148 66.1416 0)
-      (effects (font (size 1.27 1.27)) (justify left) hide)
-    )
-    (property "Value" "STB33N65M2" (at 168.148 68.453 0)
-      (effects (font (size 1.27 1.27)) (justify left) hide)
+      (effects (font (size 1.27 1.27)) (justify left))
+    )
+    (property "Value" "STP80NF70" (at 168.148 68.453 0)
+      (effects (font (size 1.27 1.27)) (justify left))
     )
     (property "Footprint" "Package_TO_SOT_THT:TO-262-3_Vertical" (at 168.275 69.215 0)
@@
     (in_bom yes) (on_board yes) (dnp no)
     (property "Reference" "Q3" (at 107.442 151.8666 0)
-      (effects (font (size 1.27 1.27)) (justify left) hide)
-    )
-    (property "Value" "STB33N65M2" (at 107.442 154.178 0)
-      (effects (font (size 1.27 1.27)) (justify left) hide)
+      (effects (font (size 1.27 1.27)) (justify left))
+    )
+    (property "Value" "STP80NF70" (at 107.442 154.178 0)
+      (effects (font (size 1.27 1.27)) (justify left))
     )
     (property "Footprint" "Package_TO_SOT_THT:TO-262-3_Vertical" (at 107.315 154.94 0)
@@
       (effects (font (size 1.27 1.27)) (justify right))
     )
-    (property "Value" "STTH2002D" (at 118.745 46.355 90)
+    (property "Value" "STTH20R04D" (at 118.745 46.355 90)
       (effects (font (size 1.27 1.27)) (justify right))
     )
@@
       (effects (font (size 1.27 1.27)) hide)
     )
-    (pin "1")
-    (pin "2")
-    (pin "3")
-    (instances
-      (project "Neonest_V_1.3"
+    (pin "3")
+    (pin "1")
+    (pin "2")
+    (instances
+      (project "Neonest_V_1.3"

Commit message: Minor changes, generated gerber files and submitted
Parts:
- R20: value 0R -> 2R2; footprint Resistor_SMD:R_0603_1608Metric -> Resistor_THT:R_Axial_DIN0204_L3.6mm_D1.6mm_P7.62mm_Horizontal
Changed lines of the file:
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@@
       (effects (font (size 1.27 1.27)) (justify left))
     )
-    (property "Value" "0R" (at 103.2764 141.097 0)
+    (property "Value" "2R2" (at 103.2764 141.097 0)
       (effects (font (size 1.27 1.27)) (justify left))
     )
-    (property "Footprint" "Resistor_SMD:R_0603_1608Metric" (at 104.775 142.24 0)
+    (property "Footprint" "Resistor_THT:R_Axial_DIN0204_L3.6mm_D1.6mm_P7.62mm_Horizontal" (at 104.775 142.24 0)
       (effects (font (size 1.27 1.27)) hide)
     )
